Commit message: 

File: gripper_control/urdf/gripper_v0/lcgripper.urdf.xacro (robot description, xacro)
@@ -98,5 +98,5 @@
       <child link="${side}_gripper_l_finger_link"/>
       <origin rpy="0 1.4224433403753787 0" xyz="-0.01750 0.0 0.053"/>
-     <limit effort="300.0" velocity = "10000" lower = "${-gripper_max_angle}" upper = "${gripper_max_angle}"/>
+     <limit effort="300.0" velocity = "10000" lower = "0" upper = "${gripper_max_angle}"/>
       <safety_controller k_position="100" k_velocity="1" soft_lower_limit = "0" soft_upper_limit = "1.4224433403753787"/>
       <axis xyz="0 1 0"/>
@@ -291,6 +291,6 @@
       <axis xyz="0 1 0" />
       <dynamics damping="${gripper_damping}" />
-      <limit effort="1000.0" velocity="0.2" lower="0.0" upper="0.135" />
-      <safety_controller k_velocity="5000.0" k_position="20.0" soft_lower_limit="${0.0-0.01}" soft_upper_limit="${0.135-0.002}" />
+      <limit effort="1000.0" velocity="0.2" lower="0.0" upper="0.15" />
+      <safety_controller k_velocity="5000.0" k_position="20.0" soft_lower_limit="${0.0}" soft_upper_limit="${0.135+0.002}" /> -->
     </joint>
     <xacro:pr2_lcgripper_finger_gazebo_v0 prefix="l" reflect="${reflect}" />

Commit message: Updated URDF with better joint definitions (follows convention everywhere) and new STL meshes. Updated transmission to accomodate URDF changes, and adds torque capping. Updated controller to do holding torque.

File: gripper_control/urdf/gripper_v0/lcgripper.urdf.xacro (robot description, xacro)
@@ -20,5 +20,5 @@
       <visual>
         <geometry>
-          <mesh filename="package://gripper_control/meshes/gripper_actuator.stl"/>
+          <mesh filename="package://gripper_control/meshes/lcg_actuator_mesh_vF.STL"/>
         </geometry>
         <origin rpy="0 0 0" xyz="0.0 0.0 0.0"/>
@@ -29,7 +29,7 @@
       <collision>
         <geometry>
-          <mesh filename="package://gripper_control/meshes/gripper_actuator.stl"/>
-        </geometry>
-        <origin rpy="0 0 0" xyz="0.0 0 0"/>
+          <mesh filename="package://gripper_control/meshes/lcg_actuator_mesh_vF.STL"/>
+        </geometry>
+        <origin rpy="0 0 0" xyz="0.0 0.0 0.0"/>
       </collision>
       <inertial>
@@ -43,12 +43,12 @@
       <child link="${side}_gripper_base_link"/>
       <!--<insert_block name="origin"/>-->
-      <origin xyz="0.03 0.0 0.0" rpy="${M_PI/2.0} 0.0 ${M_PI/2.0}"/>
+      <origin xyz="0.03 0.0 0.0" rpy="0.0 0.0 0.0"/>
     </joint>
     <link name="${side}_gripper_palm_link">
       <visual>
         <geometry>
-          <mesh filename="package://gripper_control/meshes/palm.stl"/>
-        </geometry>
-        <origin rpy="0 0 0" xyz="0.00 0.0 0.00"/>
+          <mesh filename="package://gripper_control/meshes/lcg_palm_mesh_v1-55.STL"/>
+        </geometry>
+        <origin rpy="0 0 0" xyz="0.0 0.0 0.0"/>
         <material name="${side}_palm-11_color">
           <color rgba="0.796078 0.823529 0.937255 1"/>
@@ -57,7 +57,7 @@
       <collision>
         <geometry>
-          <mesh filename="package://gripper_control/meshes/palm.stl"/>
-        </geometry>
-        <origin rpy="0 0 0" xyz="0 0 0"/>
+          <mesh filename="package://gripper_control/meshes/lcg_palm_mesh_v1-55.STL"/>
+        </geometry>
+        <origin rpy="0 0 0" xyz="0.0 0.0 0.0"/>
       </collision>
       <inertial>
@@ -70,10 +70,10 @@
       <parent link="${side}_gripper_base_link"/>
       <child link="${side}_gripper_palm_link"/>
-      <origin xyz="0.0 0.0 0.052" rpy="0 0 0"/>
+      <origin xyz="0.105 0.0 0.0" rpy="0 0 0"/>
     </joint>
     <link name="${side}_gripper_l_finger_link">
       <visual>
         <geometry>
-          <mesh filename="package://gripper_control/meshes/proximal.stl"/>
+          <mesh filename="package://gripper_control/meshes/lcg_proximal_mesh_v1-55.STL"/>
         </geometry>
         <origin rpy="0 0 0" xyz="0 0 0"/>
@@ -84,5 +84,5 @@
       <collision>
         <geometry>
-          <mesh filename="package://gripper_control/meshes/proximal.stl"/>
+          <mesh filename="package://gripper_control/meshes/lcg_proximal_mesh_v1-55.STL"/>
         </geometry>
         <origin rpy="0 0 0" xyz="0 0 0"/>
@@ -97,8 +97,8 @@
       <parent link="${side}_gripper_palm_link"/>
       <child link="${side}_gripper_l_finger_link"/>
-      <origin rpy="0 1.4224433403753787 0" xyz="-0.01750 0.0 0.053"/>
+      <origin rpy="0 0 -${M_PI/2.0}" xyz="0 -0.01750 0.0"/>
      <limit effort="300.0" velocity = "10000" lower = "0" upper = "${gripper_max_angle}"/>
       <safety_controller k_position="100" k_velocity="1" soft_lower_limit = "0" soft_upper_limit = "1.4224433403753787"/>
-      <axis xyz="0 1 0"/>
+      <axis xyz="0 0 1"/>
       <dynamics damping="0.01"/>
     </joint>
@@ -106,5 +106,5 @@
       <visual>
         <geometry>
-          <mesh filename="package://gripper_control/meshes/distal.stl"/>
+          <mesh filename="package://gripper_control/meshes/lcg_distal_mesh_v1-55.STL"/>
         </geometry>
         <origin rpy="0 0 0" xyz="0 0 0"/>
@@ -115,5 +115,5 @@
       <collision>
         <geometry>
-          <mesh filename="package://gripper_control/meshes/distal.stl"/>
+          <mesh filename="package://gripper_control/meshes/lcg_distal_mesh_v1-55.STL"/>
         </geometry>
         <origin rpy="0 0 0" xyz="0 0 0"/>
@@ -129,8 +129,8 @@
       <child link="${side}_gripper_l_finger_tip_link"/>
       <mimic joint="${side}_gripper_l_finger_joint" multiplier="-1" offset="0"/>
-      <origin rpy="0 -1.4224433403753787 0" xyz="-0.05638 0.0 0.02052"/>
+      <origin rpy="0 0 ${M_PI/2.0}" xyz="0.060 0 0"/>
       <limit effort="300.0" velocity = "10000" lower = "${-gripper_max_angle}" upper = "${gripper_max_angle}"/>
       <safety_controller k_position="100" k_velocity="1" soft_lower_limit = "0" soft_upper_limit = "1.4224433403753787"/>
-      <axis xyz="0 -1 0"/>
+      <axis xyz="0 0 -1"/>
       <dynamics damping="0.01"/>
     </joint>
@@ -138,7 +138,7 @@
       <visual>
         <geometry>
-          <mesh filename="package://gripper_control/meshes/proximal.stl"/>
-        </geometry>
-        <origin rpy="0 0 3.14159" xyz="0 0 0"/>
+          <mesh filename="package://gripper_control/meshes/lcg_proximal_mesh_v1-55.STL"/>
+        </geometry>
+        <origin rpy="0 0 0" xyz="0 0 0"/>
         <material name="${side}_gripper_r_finger-11_color">
           <color rgba="1.0 0.0 0.0 1"/>
@@ -147,7 +147,7 @@
       <collision>
         <geometry>
-          <mesh filename="package://gripper_control/meshes/proximal.stl"/>
-        </geometry>
-        <origin rpy="0 0 3.14159" xyz="0 0 0"/>
+          <mesh filename="package://gripper_control/meshes/lcg_proximal_mesh_v1-55.STL"/>
+        </geometry>
+        <origin rpy="0 0 0" xyz="0 0 0"/>
       </collision>
       <inertial>
@@ -161,8 +161,8 @@
       <child link="${side}_gripper_r_finger_link"/>
       <mimic joint="${side}_gripper_l_finger_joint" multiplier="1" offset="0"/>
-      <origin rpy="0 -1.4224433403753787 0" xyz="0.01750 0.0 0.053"/>
+      <origin rpy="0 ${M_PI} -${M_PI/2.0}" xyz="0 0.0175 0"/>
      <limit effort="300.0" velocity = "10000" lower = "${-gripper_max_angle}" upper = "${gripper_max_angle}"/>
       <safety_controller k_position="100" k_velocity="1" soft_lower_limit = "0" soft_upper_limit = "1.4224433403753787"/>
-      <axis xyz="0 1 0"/>
+      <axis xyz="0 0 1"/>
       <dynamics damping="0.01"/>
     </joint>
@@ -170,7 +170,7 @@
       <visual>
         <geometry>
-          <mesh filename="package://gripper_control/meshes/distal.stl"/>
-        </geometry>
-        <origin rpy="0 0 3.14159" xyz="0 0 0"/>
+          <mesh filename="package://gripper_control/meshes/lcg_distal_mesh_v1-55.STL"/>
+        </geometry>
+        <origin rpy="0 0 0" xyz="0 0 0"/>
         <material name="${side}_r_finger_tip-11_color">
           <color rgba="0.796078 0.823529 0.937255 1"/>
@@ -179,7 +179,7 @@
       <collision>
         <geometry>
-          <mesh filename="package://gripper_control/meshes/distal.stl"/>
-        </geometry>
-        <origin rpy="0 0 3.14159" xyz="0 0 0"/>
+          <mesh filename="package://gripper_control/meshes/lcg_distal_mesh_v1-55.STL"/>
+        </geometry>
+        <origin rpy="0 0 0" xyz="0 0 0"/>
       </collision>
       <inertial>
@@ -193,14 +193,13 @@
       <child link="${side}_gripper_r_finger_tip_link"/>
       <mimic joint="${side}_gripper_l_finger_joint" multiplier="-1" offset="0"/>
-      <origin rpy="0 1.4224433403753787 0" xyz="0.05638 0.0 0.02052"/>
+      <origin rpy="0 0 ${M_PI/2.0}" xyz="0.060 0 0"/>
       <limit effort="300.0" velocity = "10000" lower = "${-gripper_max_angle}" upper = "${gripper_max_angle}"/>
       <safety_controller k_position="100" k_velocity="1" soft_lower_limit = "0" soft_upper_limit = "1.4224433403753787"/>
-      <axis xyz="0 -1 0"/>
+      <axis xyz="0 0 -1"/>
       <dynamics damping="0.01"/>
     </joint>
     <link name="${side}_gripper_l_finger_tip_frame"/>
     <link name="${side}_gripper_tool_frame">
-      <!--
-      <visual>
+      <!--<visual>
         <geometry>
           <sphere radius="0.003"/>
@@ -210,6 +209,5 @@
           <color rgba="0.796078 0.823529 0.937255 1"/>
         </material>
-      </visual>
-      -->
+      </visual>-->
       <inertial>
         <mass value="0.1"/>
@@ -232,6 +230,6 @@
                   izz="0.001" />
       </inertial>
-      <!-- for debugging only
-      <visual>
+      <!-- for debugging only -->
+      <!--<visual>
         <origin xyz="0 0 0" rpy="0 0 0" />
         <geometry>
@@ -244,6 +242,5 @@
           <box size="0.05 0.01 0.05" />
         </geometry>
-      </collision>
-      -->
+      </collision>-->
     </link>
     <gazebo reference="${side}_gripper_motor_slider_link">
@@ -265,6 +262,6 @@
                   izz="0.0001" />
       </inertial>
-      <!-- for debugging only
-      <visual>
+      <!-- for debugging only -->
+<!--      <visual>
         <origin xyz="0 0 0" rpy="0 0 0" />
         <geometry>
@@ -277,6 +274,5 @@
           <box size="0.05 0.01 0.05" />
         </geometry>
-      </collision>
-      -->
+      </collision> -->
     </link>
     <gazebo reference="${side}_gripper_screw_link">
@@ -307,22 +303,22 @@
       screw_efficiency="${1.0}"
       screw_lead="${0.00325}"
-      j0x="${-35.0}"
+      j0x="${-0.0350}"
       j0y="${0.0}"
-      j1x="${-60.0}"
+      j1x="${-0.060}"
       j1y="${0.0}"
-      p0x="${-25.0}"
-      p0y="${2.0}"
-      p1x="${-45.0}"
-      p1y="${4.0}"
-      p2x="${-8.4}"
-      p2y="${2.3}"
-      p3x="${-44.0}"
-      p3y="${-5.0}"
-      l0="${35.0}"
-      l1="${60.0}"
-      l2="${50.0}"
-      p0_radius="${4.0}"
-      j1_radius="${3.2}"
-      thickness="${6.0}"
+      p0x="${-0.025}"
+      p0y="${0.002}"
+      p1x="${-0.045}"
+      p1y="${0.004}"
+      p2x="${-0.0084}"
+      p2y="${0.0023}"
+      p3x="${-0.044}"
+      p3y="${-0.005}"
+      l0="${0.035}"
+      l1="${0.060}"
+      l2="${0.050}"
+      p0_radius="${0.004}"
+      j1_radius="${0.0032}"
+      thickness="${0.006}"
       theta_open="${20.0}"
       theta_closed="${101.5}"

Commit message: Corrected gripper joint definitions. Positive angle on each means the joint closes. Previously this applied to proximal joints, but positive angle on the distal joints would open the link to keep the two distal links parallel.

File: gripper_control/urdf/gripper_v0/lcgripper.urdf.xacro (robot description, xacro)
@@ -132,5 +132,5 @@
       <limit effort="300.0" velocity = "10000" lower = "${-gripper_max_angle}" upper = "${gripper_max_angle}"/>
       <safety_controller k_position="100" k_velocity="1" soft_lower_limit = "0" soft_upper_limit = "1.4224433403753787"/>
-      <axis xyz="0 0 -1"/>
+      <axis xyz="0 0 1"/>
       <dynamics damping="0.01"/>
     </joint>
@@ -196,5 +196,5 @@
       <limit effort="300.0" velocity = "10000" lower = "${-gripper_max_angle}" upper = "${gripper_max_angle}"/>
       <safety_controller k_position="100" k_velocity="1" soft_lower_limit = "0" soft_upper_limit = "1.4224433403753787"/>
-      <axis xyz="0 0 -1"/>
+      <axis xyz="0 0 1"/>
       <dynamics damping="0.01"/>
     </joint>
