Commit message: Remove unused params in lcgripper xacros

File: gripper_control/urdf/gripper_v0/lcgripper.transmission.xacro (robot description, xacro)
@@ -7,5 +7,5 @@
   <xacro:macro name="pr2_lcgripper_transmission_v0" params=     "side
                                                                 gear_reduction gear_efficiency
-                                                                screw_reduction screw_efficiency screw_lead
+                                                                screw_efficiency screw_lead
                                                                 j0x j0y
                                                                 j1x j1y
@@ -36,5 +36,4 @@
                       gear_reduction="${gear_reduction}"
                       gear_efficiency="${gear_efficiency}"
-                      screw_reduction="${screw_reduction}"
                       screw_efficiency="${screw_efficiency}"
                       screw_lead="${screw_lead}"

File: gripper_control/urdf/gripper_v0/lcgripper_combined.urdf.xacro (robot description, xacro)
@@ -16,5 +16,5 @@
   <property name="lcg_palm_to_finger_x"           value="0.0587955" />
   <property name="lcg_palm_origin_offset"         value="0.053" />
-  <xacro:macro name="pr2_lcgripper_v0" params="side reflect parent *origin gear_ratio theta0 phi0 t0 L0 h a b r">
+  <xacro:macro name="pr2_lcgripper_v0" params="side reflect parent *origin">
     <link name="${side}_gripper_palm_link">
       <visual>

File: gripper_control/urdf/pr2.urdf.xacro (robot description, xacro)
@@ -111,15 +111,5 @@
     <origin xyz="0 0 0" rpy="0 0 0" />
   </xacro:pr2_forearm_v0>
-  <xacro:pr2_lcgripper_v0 reflect="1.0" side="l" parent="l_wrist_roll_link"
-               screw_reduction="${4.0/1000.0}"
-               gear_ratio="${(729.0/25.0)*(22.0/16.0)}"
-               theta0="${3.6029*M_PI/180.0}"
-               phi0="${29.7089*M_PI/180.0}"
-               t0="${-0.1914/1000.0}"
-               L0="${37.5528/1000.0}"
-               h="${0.0/1000.0}"
-               a="${68.3698/1000.0}"
-               b="${43.3849/1000.0}"
-               r="${91.5/1000.0}" >
+  <xacro:pr2_lcgripper_v0 reflect="1.0" side="l" parent="l_wrist_roll_link">
     <origin xyz="0 0 0" rpy="0 0 0" />
   </xacro:pr2_lcgripper_v0>

Commit message: Put second velo gripper on PR2 to replace standard gripper.

File: gripper_control/urdf/gripper_v0/lcgripper.transmission.xacro (robot description, xacro)
@@ -32,5 +32,5 @@
     <!-- gazebo_mimic_pid is for sim only.                                                   -->
     <transmission type="gripper_control/LCGripperTransmission" name="${side}_gripper_trans" >
-      <actuator       name="${side}_gripper_motor" />
+      <actuator       name="${side}_velo_gripper_motor" />
       <gap_joint      name="${side}_gripper_joint"
                       gear_reduction="${gear_reduction}"

File: gripper_control/urdf/pr2.urdf.xacro (robot description, xacro)
@@ -91,17 +91,7 @@
     <origin xyz="0 0 0" rpy="0 0 0" />
   </xacro:pr2_forearm_v0>
-  <xacro:pr2_gripper_v0 reflect="-1.0" side="r" parent="r_wrist_roll_link"
-               screw_reduction="${4.0/1000.0}"
-               gear_ratio="${(729.0/25.0)*(22.0/16.0)}"
-               theta0="${3.6029*M_PI/180.0}"
-               phi0="${29.7089*M_PI/180.0}"
-               t0="${-0.1914/1000.0}"
-               L0="${37.5528/1000.0}"
-               h="${0.0/1000.0}"
-               a="${68.3698/1000.0}"
-               b="${43.3849/1000.0}"
-               r="${91.5/1000.0}" >
-    <origin xyz="0 0 0" rpy="0 0 0" />
-  </xacro:pr2_gripper_v0>
+  <xacro:pr2_lcgripper_v0 reflect="1.0" side="r" parent="r_wrist_roll_link">
+     <origin xyz="0.135 0.0 0.0" rpy="0 0 0"/>
+  </xacro:pr2_lcgripper_v0>
   <xacro:pr2_shoulder_v0 side="l" reflect="1" parent="torso_lift_link">
     <origin xyz="0.0 0.188 0.0" rpy="0 0 0" />
