Commit message: Remove lcgripper param screw_reduction. Change ParamServer to ParamFetcher. Less formal. Calibration mode of transmission will convert to/from ballscrew position/force. Remove some commented-out deprecated methods Use MACROS for RAD2REV, REV2DEG, DEG2REV, REV2DEG Remove trailing whitespace

File: gripper_control/urdf/gripper_v0/lcgripper_combined.urdf.xacro (robot description, xacro)
@@ -16,5 +16,5 @@
   <property name="lcg_palm_to_finger_x"           value="0.0587955" />
   <property name="lcg_palm_origin_offset"         value="0.053" />
-  <xacro:macro name="pr2_lcgripper_v0" params="side reflect parent *origin gear_ratio screw_reduction theta0 phi0 t0 L0 h a b r">
+  <xacro:macro name="pr2_lcgripper_v0" params="side reflect parent *origin gear_ratio theta0 phi0 t0 L0 h a b r">
     <link name="${side}_gripper_palm_link">
       <visual>
@@ -274,5 +274,4 @@
       screw_efficiency="${1.0}"
       screw_lead="${0.00325}"
-      screw_reduction="${1/0.00325}"
       j0x="${-0.0350}"
       j0y="${0.0}"

Commit message: Mostly working on PR2.  Try new capped_pos. engine.

File: gripper_control/urdf/gripper_v0/lcgripper_combined.urdf.xacro (robot description, xacro)
@@ -263,6 +263,6 @@
       <axis xyz="0 1 0" />
       <dynamics damping="${gripper_damping}" />
-      <limit effort="1000.0" velocity="0.2" lower="0.0" upper="0.15" />
-      <safety_controller k_velocity="5000.0" k_position="20.0" soft_lower_limit="${0.0}" soft_upper_limit="${0.135+0.002}" /> -->
+    <limit effort="333.3" lower="-99999.9" upper="99999.9" velocity="9.9"/>
+    <safety_controller k_position="1e6" k_velocity="1e6" soft_lower_limit="-99999.1" soft_upper_limit="99999.1"/>
     </joint>
     <xacro:pr2_lcgripper_finger_gazebo_v0 prefix="l" reflect="${reflect}" />

Commit message: fixes bug for the gripper xacro to use the origin param

File: gripper_control/urdf/gripper_v0/lcgripper_combined.urdf.xacro (robot description, xacro)
@@ -42,5 +42,5 @@
       <parent link="${parent}"/>
       <child link="${side}_gripper_palm_link"/>
-      <origin xyz="0.135 0.0 0.0" rpy="0 0 0"/>
+      <insert_block name="origin" />
     </joint>
     <link name="${side}_gripper_l_finger_link">

File: gripper_control/urdf/pr2.urdf.xacro (robot description, xacro)
@@ -112,5 +112,5 @@
   </xacro:pr2_forearm_v0>
   <xacro:pr2_lcgripper_v0 reflect="1.0" side="l" parent="l_wrist_roll_link">
-    <origin xyz="0 0 0" rpy="0 0 0" />
+     <origin xyz="0.135 0.0 0.0" rpy="0 0 0"/>
   </xacro:pr2_lcgripper_v0>
   <!-- Forearm cam Position is a guess, based on full robot calibration -->

Commit message: Remove gap_to_effective_dist_coeffs_ and use virtual work instead.  Comment-out extensor spring force.  Comment-out safety controllers on passive links.

File: gripper_control/urdf/gripper_v0/lcgripper_combined.urdf.xacro (robot description, xacro)
@@ -66,10 +66,12 @@
       </inertial>
     </link>
-    <joint name="${side}_gripper_l_finger_joint" type="revolute">
+    <joint name="${side}_gripper_l_finger_joint" type="continuous">
       <parent link="${side}_gripper_palm_link"/>
       <child link="${side}_gripper_l_finger_link"/>
       <origin rpy="0 0 -${M_PI/2.0}" xyz="0 -0.01750 0.0"/>
+<!--
      <limit effort="300.0" velocity = "10000" lower = "0" upper = "${gripper_max_angle}"/>
       <safety_controller k_position="100" k_velocity="1" soft_lower_limit = "0" soft_upper_limit = "1.4224433403753787"/>
+-->
       <axis xyz="0 0 1"/>
       <dynamics damping="0.01"/>
@@ -97,11 +99,13 @@
       </inertial>
     </link>
-    <joint name="${side}_gripper_l_finger_tip_joint" type="revolute">
+    <joint name="${side}_gripper_l_finger_tip_joint" type="continuous">
       <parent link="${side}_gripper_l_finger_link"/>
       <child link="${side}_gripper_l_finger_tip_link"/>
       <mimic joint="${side}_gripper_l_finger_joint" multiplier="-1" offset="0"/>
       <origin rpy="0 0 ${M_PI/2.0}" xyz="0.060 0 0"/>
+<!--
       <limit effort="300.0" velocity = "10000" lower = "${-gripper_max_angle}" upper = "${gripper_max_angle}"/>
       <safety_controller k_position="100" k_velocity="1" soft_lower_limit = "0" soft_upper_limit = "1.4224433403753787"/>
+-->
       <axis xyz="0 0 1"/>
       <dynamics damping="0.01"/>
@@ -129,11 +133,13 @@
       </inertial>
     </link>
-    <joint name="${side}_gripper_r_finger_joint" type="revolute">
+    <joint name="${side}_gripper_r_finger_joint" type="continuous">
       <parent link="${side}_gripper_palm_link"/>
       <child link="${side}_gripper_r_finger_link"/>
       <mimic joint="${side}_gripper_l_finger_joint" multiplier="1" offset="0"/>
       <origin rpy="0 ${M_PI} -${M_PI/2.0}" xyz="0 0.0175 0"/>
+<!--
      <limit effort="300.0" velocity = "10000" lower = "${-gripper_max_angle}" upper = "${gripper_max_angle}"/>
       <safety_controller k_position="100" k_velocity="1" soft_lower_limit = "0" soft_upper_limit = "1.4224433403753787"/>
+-->
       <axis xyz="0 0 1"/>
       <dynamics damping="0.01"/>
@@ -161,12 +167,13 @@
       </inertial>
     </link>
-    <joint name="${side}_gripper_r_finger_tip_joint" type="revolute">
+    <joint name="${side}_gripper_r_finger_tip_joint" type="continuous">
       <parent link="${side}_gripper_r_finger_link"/>
       <child link="${side}_gripper_r_finger_tip_link"/>
       <mimic joint="${side}_gripper_l_finger_joint" multiplier="-1" offset="0"/>
       <origin rpy="0 0 ${M_PI/2.0}" xyz="0.060 0 0"/>
+<!--
       <limit effort="300.0" velocity = "10000" lower = "${-gripper_max_angle}" upper = "${gripper_max_angle}"/>
       <safety_controller k_position="100" k_velocity="1" soft_lower_limit = "0" soft_upper_limit = "1.4224433403753787"/>
-      <axis xyz="0 0 1"/>
+-->
       <dynamics damping="0.01"/>
     </joint>
@@ -224,5 +231,7 @@
       <parent link="${side}_gripper_palm_link"/>
       <child link="${side}_gripper_motor_slider_link"/>
+<!--
       <limit effort="1000.0" velocity="0.2" lower="-0.135" upper="0.135" />
+-->
     </joint>
     <link name="${side}_gripper_motor_screw_link">
