Commit message: Updated full PR2 URDF with Jon's calibrated one.

File: gripper_control/urdf/pr2.urdf.xacro (robot description, xacro)
@@ -3,5 +3,5 @@
        xmlns:controller="http://playerstage.sourceforge.net/gazebo/xmlschema/#controller"
        xmlns:interface="http://playerstage.sourceforge.net/gazebo/xmlschema/#interface"
-       xmlns:xacro="http://playerstage.sourceforge.net/gazebo/xmlschema/#interface"
+       xmlns:xacro="http://www.ros.org/wiki/xacro"
        name="pr2" >
   <!-- The following included files set up definitions of parts of the robot body -->
@@ -25,4 +25,5 @@
   <!-- Head sensors -->
   <include filename="$(find pr2_description)/urdf/sensors/head_sensor_package.urdf.xacro" />
+  <include filename="$(find pr2_description)/urdf/sensors/kinect_prosilica_camera.urdf.xacro" />
   <!-- Camera sensors -->
   <include filename="$(find pr2_description)/urdf/sensors/wge100_camera.urdf.xacro" />
@@ -61,6 +62,22 @@
   <xacro:projector_wg6802418_v0 name="projector_wg6802418" parent="head_plate_frame" >
     <!-- Camera is slightly recessed from front, where is camera origin? Lens? -->
-    <origin xyz="0.046457 0.110 0.0546" rpy="0 0 0" />
+    <origin xyz="0 0.110 0.0546" rpy="0 0 0" />
   </xacro:projector_wg6802418_v0>
+  <!-- Base of Kinect/Prosilica Mount -->
+  <xacro:kinect_prosilica_camera_swept_back_v0 name="head_mount" parent="head_plate_frame" >
+    <origin xyz="-0.137376 0 0.091746" rpy="0 0 0" />
+    <!--
+          Was -0.1 0 0.09225, -0.138 0 0.09225 looks good front back and sheet metal on bolt pattern,
+          -0.138 0 0.06225 is where Prosilica FOV just clears the head.
+          This is 30 mm (!) below the position in SolidWorks.
+          Lowering the Prosilica by this amount in SW makes the FOV hit around the aluminum / plastic junction.
+          Turns out that head_plate_frame is in some random position in space.
+          It is [0.0232 0 0.0645 from its parent, head_tilt_link.
+          The distance from head_plate_frame to the head_kinect_prosilica is 137.376 mm X and 91.746 mm Z.
+          So the origin should in fact be -0.137376 0 0.091746.
+          John is changing the Prosilica FOV based on my numbers.
+          Just need to roscd and svn up.
+    -->
+  </xacro:kinect_prosilica_camera_swept_back_v0>
   <xacro:pr2_tilting_laser_v0 name="laser_tilt" parent="torso_lift_link" laser_calib_ref="0.0">
     <origin xyz="0.09893 0 0.227" rpy="0 0 0" />
