Commit message: trying to commit more changes

File: velo_description/urdf/velo_v0/velo.urdf.xacro (robot description, xacro)
@@ -5,6 +5,6 @@
        xmlns:interface="http://playerstage.sourceforge.net/gazebo/xmlschema/#interface"
        xmlns:xacro="http://ros.org/wiki/xacro">
-  <include filename="$(find gripper_control)/urdf/gripper_v0/lcgripper.gazebo.xacro" />
-  <include filename="$(find gripper_control)/urdf/gripper_v0/lcgripper.transmission.xacro" />
+  <include filename="$(find velo_description)/urdf/velo_v0/velo.gazebo.xacro" />
+  <include filename="$(find velo_description)/urdf/velo_v0/velo.transmission.xacro" />
   <property name="M_PI" value="3.1415926535897931" />
   <property name="gripper_max_angle" value="1.4224433403753787" />
@@ -20,5 +20,5 @@
       <visual>
         <geometry>
-          <mesh filename="package://gripper_control/meshes/lcg_actuator_palm_mesh_v1-55.STL"/>
+          <mesh filename="package://velo_description/meshes/velo_actuator_palm_mesh_v1-55.STL"/>
         </geometry>
         <origin rpy="0 0 0" xyz="0.0 0.0 0.0"/>
@@ -29,5 +29,5 @@
       <collision>
         <geometry>
-          <mesh filename="package://gripper_control/meshes/lcg_actuator_palm_mesh_v1-55.STL"/>
+          <mesh filename="package://velo_description/meshes/velo_actuator_palm_mesh_v1-55.STL"/>
         </geometry>
         <origin rpy="0 0 0" xyz="0.0 0.0 0.0"/>
@@ -47,5 +47,5 @@
       <visual>
         <geometry>
-          <mesh filename="package://gripper_control/meshes/lcg_proximal_mesh_v1-55.STL"/>
+          <mesh filename="package://velo_description/meshes/velo_proximal_mesh_v1-55.STL"/>
         </geometry>
         <origin rpy="0 0 0" xyz="0 0 0"/>
@@ -56,5 +56,5 @@
       <collision>
         <geometry>
-          <mesh filename="package://gripper_control/meshes/lcg_proximal_mesh_v1-55.STL"/>
+          <mesh filename="package://velo_description/meshes/velo_proximal_mesh_v1-55.STL"/>
         </geometry>
         <origin rpy="0 0 0" xyz="0 0 0"/>
@@ -80,5 +80,5 @@
       <visual>
         <geometry>
-          <mesh filename="package://gripper_control/meshes/lcg_distal_mesh_v1-55.STL"/>
+          <mesh filename="package://velo_description/meshes/velo_distal_mesh_v1-55.STL"/>
         </geometry>
         <origin rpy="0 0 0" xyz="0 0 0"/>
@@ -89,5 +89,5 @@
       <collision>
         <geometry>
-          <mesh filename="package://gripper_control/meshes/lcg_distal_mesh_v1-55.STL"/>
+          <mesh filename="package://velo_description/meshes/velo_distal_mesh_v1-55.STL"/>
         </geometry>
         <origin rpy="0 0 0" xyz="0 0 0"/>
@@ -114,5 +114,5 @@
       <visual>
         <geometry>
-          <mesh filename="package://gripper_control/meshes/lcg_proximal_mesh_v1-55.STL"/>
+          <mesh filename="package://velo_description/meshes/velo_proximal_mesh_v1-55.STL"/>
         </geometry>
         <origin rpy="0 0 0" xyz="0 0 0"/>
@@ -123,5 +123,5 @@
       <collision>
         <geometry>
-          <mesh filename="package://gripper_control/meshes/lcg_proximal_mesh_v1-55.STL"/>
+          <mesh filename="package://velo_description/meshes/velo_proximal_mesh_v1-55.STL"/>
         </geometry>
         <origin rpy="0 0 0" xyz="0 0 0"/>
@@ -148,5 +148,5 @@
       <visual>
         <geometry>
-          <mesh filename="package://gripper_control/meshes/lcg_distal_mesh_v1-55.STL"/>
+          <mesh filename="package://velo_description/meshes/velo_distal_mesh_v1-55.STL"/>
         </geometry>
         <origin rpy="0 0 0" xyz="0 0 0"/>
@@ -157,5 +157,5 @@
       <collision>
         <geometry>
-          <mesh filename="package://gripper_control/meshes/lcg_distal_mesh_v1-55.STL"/>
+          <mesh filename="package://velo_description/meshes/velo_distal_mesh_v1-55.STL"/>
         </geometry>
         <origin rpy="0 0 0" xyz="0 0 0"/>

File: velo_pr2/urdf/pr2.urdf.xacro (robot description, xacro)
@@ -14,5 +14,6 @@
   <!-- PR2 gripper -->
   <include filename="$(find pr2_description)/urdf/gripper_v0/gripper.urdf.xacro" />
-  <include filename="$(find gripper_control)/urdf/gripper_v0/lcgripper_combined.urdf.xacro" />
+  <!-- Velo gripper -->
+  <include filename="$(find velo_description)/urdf/velo_v0/velo.urdf.xacro" />
   <!-- PR2 head -->
   <include filename="$(find pr2_description)/urdf/head_v0/head.urdf.xacro" />
